Commit message: Update actuator_description.urdf
puse el link world para que el robot quede fijo en el piso :)

File: third_pkg/urdf/actuator_description.urdf (robot description, URDF)
Before this commit: robot actuator, 3 links, 2 joints
Links:
- removed link base_link
- added link world
- link end_effector: mass 0.00071418 -> 0.4
Joints:
- removed joint base_link_motor
- added joint world_motor: type fixed, parent world, child motor
- joint motor_end_effector: limit lower=-3.14 upper=3.14 effort=2.1 velocity=10.471975512 -> lower=-3.14 upper=3.14 effort=2.1 velocity=0.5; origin xyz=0.03225 0.0 0.0135 rpy=0.0 0.0 0.0 -> xyz=0.03225 0.0 0.0140 rpy=0.0 0.0 0.0
